File: JtagArm20Adapter.kicad_sch (KiCad schematic)
At the start: 8 parts, among them J1 Conn_02x05_Odd_Even, J2 Conn_02x10_Odd_Even, J3 Conn_01x06, J4 Conn_02x10_Odd_Even, J5 Conn_02x03_Odd_Even

Commit message: rev 0.2
Parts:
- removed J2: Conn_02x10_Odd_Even, Connector_PinHeader_1.27mm:PinHeader_2x10_P1.27mm_Vertical_SMD, symbol Connector_Generic:Conn_02x10_Odd_Even
- removed JP1, JP2, JP3: SolderJumper_2_Open, Jumper:SolderJumper-2_P1.3mm_Open_TrianglePad1.0x1.5mm, symbol Jumper:SolderJumper_2_Open
- added C (x4): C_Small, symbol Device:C_Small
- added U (x2): (no value), symbol Device:R
- added U (x2): MCP1703A-1202_SOT23, Package_TO_SOT_SMD:SOT-23, symbol Regulator_Linear:MCP1703A-1202_SOT23
- added U: (no value), symbol Connector_Generic:Conn_02x03_Odd_Even
- added U: (no value), symbol hardware_nrf52840_pa_beacon_hat:USB_C_Receptacle_USB2.0-Connector
- U: renamed from J4; value Conn_02x10_Odd_Even -> (none); footprint Connector_PinSocket_2.54mm:PinSocket_2x10_P2.54mm_Horizontal -> (none)
- U: renamed from J1; value Conn_02x05_Odd_Even -> (none); footprint Connector_PinHeader_1.27mm:PinHeader_2x05_P1.27mm_Vertical_SMD -> (none)
- U: renamed from J3; value Conn_01x06 -> (none); footprint Connector_PinHeader_2.54mm:PinHeader_1x06_P2.54mm_Vertical -> (none)
- U: renamed from J5; value Conn_02x03_Odd_Even -> (none); footprint Connector_PinHeader_2.54mm:PinHeader_2x03_P2.54mm_Vertical_SMD -> (none)
Connections:
- net GND: now also C.2, C.2, C.2, C.2, U.1, U.1, U.1 (GND), U.1 (GND), U.A1 (GND), U.A12 (GND), U.B1 (GND), U.B12 (GND), U.S1 (SHIELD)
- net VTref: now also U.2 (Pin_2), U.4 (Pin_4), U.6 (Pin_6); no longer U.1 (Pin_1), U.1 (Pin_1), U.1 (Pin_1)
- net DBGACK: no longer names the net of U.19 (Pin_19)
- net DBGRQ: no longer names the net of U.17 (Pin_17)
- net TDI: no longer names the net of U.5 (Pin_5)
- net TDI: no longer U.8 (Pin_8)
- net nTRST: no longer names the net of U.3 (Pin_3)
- new net: U.2, U.B5 (CC2)
- new net: U.2, U.A5 (CC1)
- new net +1V8: C.1, U.2 (VO), U.5 (Pin_5)
- new net +3V3: C.1, U.2 (VO), U.3 (Pin_3)
- new net +5V: C.1, C.1, U.3 (VI), U.3 (VI), U.A4 (VBUS), U.A9 (VBUS), U.B4 (VBUS), U.B9 (VBUS)
- new net VTrefJ: U.1 (Pin_1), U.1 (Pin_1), U.1 (Pin_1), U.1 (Pin_1)
- no-connect marks 8 -> 15
